File: _autosave-pkm_agv.kicad_pcb (KiCad board)
At the start: 2 copper layers, 198.6 x 51.3 mm, 28 parts, among them J1 DRVAR, J10 ENCA, J11 ECNB, J12 ENCC, J13 ENCD, J14 BATTMTR, J15 MOTORA, J16 MOTORB, J17 MOTORC, J18 MOTORB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

Commit message: ver 1
Other:
- board text added: "ASTAR TECH"
Changed lines of the file:
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@@
   (gr_circle (center 41.275 85.852) (end 42.545 87.122)
     (stroke (width 0.1) (type default)) (fill none) (layer "Edge.Cuts"))
+  (gr_text "ASTAR TECH" (at 65.405 120.015) (layer "F.SilkS")
+    (effects (font (size 1.5 1.5) (thickness 0.3) bold) (justify left bottom))
+  )
   (segment (start 90.19 93.98) (end 128.905 93.98) (width 0.3) (layer "B.Cu") (net 1))
   (segment (start 128.905 93.98) (end 131.850834 96.925834) (width 0.3) (layer "B.Cu") (net 1))
