File: pkm_agv.kicad_sch (KiCad schematic)
At the start: 25 parts, among them J1 Conn_01x04_Socket, J10 Conn_01x04_Socket, J11 Conn_01x04_Socket, J12 Conn_01x04_Socket, J13 Conn_01x02_Socket, J2 Conn_01x04_Socket, J3 Conn_01x04_Socket, J4 Conn_01x04_Socket, J5 Conn_01x04_Socket, J6 Conn_01x04_Socket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

Commit message: ver 1
Parts:
- removed D2, D3, D4, D5: LED, symbol Device:LED
- removed J13: Conn_01x02_Socket, symbol Connector:Conn_01x02_Socket
- removed R, R2, R3, R4: 330, symbol Device:R
- removed U1: ~, symbol STM32:STM32F4_BlackPill
- added C1, C2: 10uF, Capacitor_SMD:CP_Elec_4x5.4, symbol Device:C_Polarized_Small_US
- added J14: BATTMTR, XT90PW-M:AMASS_XT90PW-M, symbol XT90PW-M:XT90PW-M
- added J15: MOTORA, TerminalBlock:TerminalBlock_bornier-2_P5.08mm, symbol Connector:Screw_Terminal_01x02
- added J16, J18: MOTORB, TerminalBlock:TerminalBlock_bornier-2_P5.08mm, symbol Connector:Screw_Terminal_01x02
- added J17: MOTORC, TerminalBlock:TerminalBlock_bornier-2_P5.08mm, symbol Connector:Screw_Terminal_01x02
- added J19: BATTMCU, XT90PW-M:AMASS_XT90PW-M, symbol XT90PW-M:XT90PW-M
- added J20: UARTCOM, Connector_PinHeader_2.54mm:PinHeader_1x03_P2.54mm_Vertical, symbol Connector:Conn_01x03_Socket
- added J21: ACTB, Connector_PinHeader_2.54mm:PinHeader_1x04_P2.54mm_Vertical, symbol Connector:Conn_01x04_Socket
- added J9: ACTA, Connector_PinHeader_2.54mm:PinHeader_1x04_P2.54mm_Vertical, symbol Connector:Conn_01x04_Socket
- added U2: AMS1117-5.0, Package_TO_SOT_SMD:SOT-223-3_TabPin2, symbol Regulator_Linear:AMS1117-5.0
- added U3: BlackPill_STLINK, BlackPill_STLINK:BlackPill_STLINK, symbol blackpill_stlink:BlackPill_STLINK
- BZ1: footprint (none) -> Buzzer_Beeper:Buzzer_15x7.5RM7.6
- D2: renamed from D1; footprint (none) -> LED_SMD:LED_1206_3216Metric_Pad1.42x1.75mm_HandSolder
- J1: value Conn_01x04_Socket -> DRVAR; footprint (none) -> Connector_PinHeader_2.54mm:PinHeader_1x04_P2.54mm_Vertical
- J10: renamed from J9; value Conn_01x04_Socket -> ENCA; footprint (none) -> Connector_PinHeader_2.54mm:PinHeader_1x04_P2.54mm_Vertical
- J11: renamed from J10; value Conn_01x04_Socket -> ECNB; footprint (none) -> Connector_PinHeader_2.54mm:PinHeader_1x04_P2.54mm_Vertical
- J12: renamed from J11; value Conn_01x04_Socket -> ENCC; footprint (none) -> Connector_PinHeader_2.54mm:PinHeader_1x04_P2.54mm_Vertical
- J13: renamed from J12; value Conn_01x04_Socket -> ENCD; footprint (none) -> Connector_PinHeader_2.54mm:PinHeader_1x04_P2.54mm_Vertical
- J2: renamed from J3; value Conn_01x04_Socket -> DRVBR; footprint (none) -> Connector_PinHeader_2.54mm:PinHeader_1x04_P2.54mm_Vertical
- J3: renamed from J5; value Conn_01x04_Socket -> DRVCR; footprint (none) -> Connector_PinHeader_2.54mm:PinHeader_1x04_P2.54mm_Vertical
- J4: renamed from J7; value Conn_01x04_Socket -> DRVDR; footprint (none) -> Connector_PinHeader_2.54mm:PinHeader_1x04_P2.54mm_Vertical
- J5: renamed from J2; value Conn_01x04_Socket -> DRVAL; footprint (none) -> Connector_PinHeader_2.54mm:PinHeader_1x04_P2.54mm_Vertical
- J6: renamed from J4; value Conn_01x04_Socket -> DRVBL; footprint (none) -> Connector_PinHeader_2.54mm:PinHeader_1x04_P2.54mm_Vertical
- J7: renamed from J6; value Conn_01x04_Socket -> DRVCL; footprint (none) -> Connector_PinHeader_2.54mm:PinHeader_1x04_P2.54mm_Vertical
- J8: value Conn_01x04_Socket -> DRVDL; footprint (none) -> Connector_PinHeader_2.54mm:PinHeader_1x04_P2.54mm_Vertical
- R2: renamed from R1; footprint (none) -> Resistor_SMD:R_1206_3216Metric_Pad1.30x1.75mm_HandSolder
Connections:
- net +5V: now also C1.1, J21.1 (Pin_1), J9.1 (Pin_1), U2.2 (VO), U3.18 (5V), U3.40 (5V)
- net Buzzer: now also U3.30 (PA4)
- net ENCL_A: now also U3.6 (PA9)
- net ENCL_B: now also U3.11 (PB3)
- net ENCL_C: now also U3.15 (PB7)
- net ENCL_D: now also U3.27 (PA1)
- net ENCR_A: now also U3.5 (PA8)
- net ENCR_B: now also U3.31 (PA5)
- net ENCR_C: now also U3.14 (PB6)
- net ENCR_D: now also U3.26 (PA0)
- net ENL_A: now also U3.37 (PB10)
- net ENL_B: now also U3.2 (PB13)
- net ENL_C: now also U3.4 (PB15)
- net ENL_D: now also U3.10 (PA15)
- net ENR_A: now also U3.36 (PB2)
- net ENR_B: now also U3.1 (PB12)
- net ENR_C: now also U3.3 (PB14)
- net ENR_D: now also U3.7 (PA10)
- net GND: now also C1.2, C2.2, J19.N (NEG), J20.3 (Pin_3), J21.4 (Pin_4), J9.4 (Pin_4), U2.1 (GND), U3.19 (GND), U3.39 (GND), U3.44 (GND)
- net PWML_A: now also U3.33 (PA7)
- net PWML_B: now also U3.35 (PB1)
- net PWML_C: now also U3.29 (PA3)
- net PWML_D: now also U3.17 (PB9)
- net PWMR_A: now also U3.32 (PA6)
- net PWMR_B: now also U3.34 (PB0)
- net PWMR_C: now also U3.28 (PA2)
- net PWMR_D: now also U3.16 (PB8)
- net UART_RX: now also J20.2 (Pin_2), U3.9 (PA12)
- net UART_TX: now also J20.1 (Pin_1), U3.8 (PA11)
- net LED_A renamed LED
- net LED: now also U3.12 (PB4)
- new net 12V_BATT: J14.P (POS), J15.1 (Pin_1), J16.1 (Pin_1), J17.1 (Pin_1), J18.1 (Pin_1)
- new net 2S_BATT: C2.1, J19.P (POS), U2.3 (VI)
- new net GND_BATT: J14.N (NEG), J15.2 (Pin_2), J16.2 (Pin_2), J17.2 (Pin_2), J18.2 (Pin_2)
- new net INA_DRVA: J9.2 (Pin_2), U3.13 (PB5)
- new net INA_DRVB: J21.2 (Pin_2), U3.23 (PC14)
- new net INB_DRVA: J9.3 (Pin_3), U3.24 (PC15)
- new net INB_DRVB: J21.3 (Pin_3), U3.22 (PC13)
- no-connect marks 12 -> 15
Other:
- note added: "BATTERY_MCU"
- note added: "BATTERY_MOTOR"
- note added: "BTS7960_Driver_A"
- note added: "BTS7960_Driver_B"
- note added: "BTS7960_Driver_C"
- note added: "BTS7960_Driver_D"
- note added: "BUZZER"
- note added: "COMMUNICATION_UART"
- note added: "DRIVER_ACT_A"
- note added: "DRIVER_ACT_B"
- note added: "ENCODER_A"
- note added: "ENCODER_B"
- note added: "ENCODER_C"
- note added: "ENCODER_D"
- note added: "LED_A"
- note added: "MOTOR_A"
- note added: "MOTOR_B"
- note added: "MOTOR_C"
- note added: "MOTOR_D"
- note added: "REGULATOR_2S"
- note added: "STM32F411CEU6"
- moved on the sheet: D2, R2
